File: STM32F103_DEMO/stm32.kicad_sch (KiCad schematic)
At the start: 28 parts, among them J1 USB_B_Micro, J2 Conn_01x04_Male, J3 Conn_01x04_Male, J4 Conn_01x04_Male, SW1 SW_SPDT, U1 AMS1117-3.3, U2 STM32F103C8T6, Y1 16MHz

Commit message: STM32F103 Board
Parts:
- added H1, H2, H3, H4: MountingHole, MountingHole:MountingHole_2.2mm_M2, symbol Mechanical:MountingHole
- C1, C2: footprint (none) -> Capacitor_SMD:C_0805_2012Metric
- C10, C11, C12, C13, C4, C5, C6, C7, C8, C9: footprint (none) -> Capacitor_SMD:C_0402_1005Metric
- C3: footprint (none) -> Capacitor_SMD:C_0603_1608Metric
- D1: footprint (none) -> LED_SMD:LED_0603_1608Metric
- FB1: footprint (none) -> Inductor_SMD:L_0603_1608Metric
- J1: footprint (none) -> Connector_USB:USB_Micro-B_Wuerth_629105150521
- J2, J3, J4: footprint (none) -> Connector_PinHeader_2.54mm:PinHeader_1x04_P2.54mm_Vertical
- R1, R2, R3, R4, R5: footprint (none) -> Resistor_SMD:R_0402_1005Metric
- SW1: footprint (none) -> Button_Switch_SMD:SW_SPDT_PCM12
- Y1: footprint (none) -> Crystal:Crystal_SMD_3225-4Pin_3.2x2.5mm
Connections:
- net +3V3: now also J2.1 (Pin_1), J4.1 (Pin_1); no longer J2.4 (Pin_4), J4.4 (Pin_4)
- net GND: now also J2.4 (Pin_4), J4.4 (Pin_4); no longer J2.1 (Pin_1), J4.1 (Pin_1)
- net I2C_SCL: now also J4.2 (Pin_2); no longer J4.3 (Pin_3)
- net I2C_SDA: now also J4.3 (Pin_3); no longer J4.2 (Pin_2)
- net USART1_RX: now also J2.3 (Pin_3); no longer J2.2 (Pin_2)
- net USART1_TX: now also J2.2 (Pin_2); no longer J2.3 (Pin_3)
Other:
- note added: "M2"
- note added: "Mounting Holes"
